Commit message: Final sonrası versiyon display.launch ile gelen gui ile robot kontrol edilebiliyor.

File: src/my_spherical_manipulator/urdf/spherical_manipulator.urdf (robot description, URDF)
Before this commit: robot spherical_manipulator, 4 links, 3 joints
Joints:
- joint base_Revolute_1: limit effort=300 velocity=1.0 -> lower=-1.57 upper=1.57 effort=300 velocity=1.0; type continuous -> revolute
- joint large_Revolute_2: limit effort=300 velocity=1.0 -> lower=-1.57 upper=1.57 effort=300 velocity=1.0; type continuous -> revolute
- joint medium_Revolute_3: limit effort=300 velocity=1.0 -> lower=-1.57 upper=1.57 effort=300 velocity=1.0; type continuous -> revolute

Commit message: stl updated version

File: src/my_spherical_manipulator/urdf/spherical_manipulator.urdf (robot description, URDF)
Before this commit: robot spherical_manipulator, 4 links, 3 joints
Links:
- added link dummy_base, mass 150.036157
- link base: mass 50.036157 -> None
Joints:
- added joint base_to_dummy: type fixed, parent base, child dummy_base, origin xyz=0 0 0 rpy=0 0 0
- joint base_Revolute_1: limit effort=300 velocity=1.0 -> lower=-1.57 upper=1.57 effort=100.0 velocity=1.0
- joint large_Revolute_2: limit effort=300 velocity=1.0 -> lower=-1.57 upper=1.57 effort=100.0 velocity=1.0
- joint medium_Revolute_3: limit effort=300 velocity=1.0 -> lower=-1.57 upper=1.57 effort=100.0 velocity=1.0
