Commit message: save commit before python script edit

File: src/spherical_arm/urdf/spherical_arm.urdf (robot description, URDF)
Before this commit: robot spherical_arm, 11 links, 10 joints
Joints:
- joint Base_Revolute: limit lower=-1.57 upper=1.57 effort=10 velocity=1 -> lower=-1.5708 upper=1.5708 effort=10 velocity=1; origin xyz=-0.011931 0.2308 -0.014931 rpy=0 0.12246 0 -> xyz=-0.011931 0.2308 -0.014931 rpy=0 +0.32246 0
- joint Revolute3: limit lower=-1.57 upper=1.57 effort=10 velocity=1 -> lower=-1.5708 upper=1.5708 effort=10 velocity=1
- joint Revolute_2: limit lower=-1.57 upper=1.57 effort=10 velocity=1 -> lower=-1.5708 upper=1.5708 effort=10 velocity=1
